File: alarmeATMEGA328/alarmeATMEGA328.sch (KiCad schematic (older format))
At the start: 10 parts

Commit message: Kicad .sch MAJ
Parts:
- added C? (x3): C, symbol C
- added C?: CP, symbol CP
- added R? (x2): R, symbol R
- added Y?: Crystal, symbol Crystal
Connections:
- net at J?.1: now also T?.1 (AA)
- net at J?.2: now also T?.2 (AB)
- net at T?.3 (SA): now also D?.2
- net at T?.4 (SB): now also D?.4
- net at D?.1 (-): now also C?.2, D?.1 (K), U?.2, U?.GND, C?.2
- net at D?.3 (+): now also C?.1, U?.VI
- net at U?.VO: now also R?.1, C?.1, R?.2
- net at R?.2: now also D?.2 (A)
- net at U?.1: now also R?.1
- net GND-ATMEGA328P: now reaches U?.3
- net GND-ATMEGA328P: now also IC?.8 (GND), C?.2
- net at U?.4: now also IC?.4 ((PCINT18/INT0)PD2), R?.2, C?.1
- net +5v-ATMEGA328P: now reaches IC?.7 (VCC)
- net +5v-ATMEGA328P: now also R?.1
Other:
- note added: "Digital PIN 2"
- moved on the sheet: C?, D?, R?, U?
Changed lines of the file:
@@
 LIBS:contrib
 LIBS:valves
+LIBS:alarmeATMEGA328-cache
 EELAYER 25 0
 EELAYER END
@@
 encoding utf-8
 Sheet 1 1
-Title ""
-Date ""
-Rev ""
+Title "Alarme ATMEGA328"
+Date "2020-05-02"
+Rev "1.0"
 Comp ""
 Comment1 ""
@@
 L CP C?
 U 1 1 5EACB486
-P 4200 2900
-F 0 "C?" H 4225 3000 50  0000 L CNN
-F 1 "CP" H 4225 2800 50  0000 L CNN
-F 2 "" H 4238 2750 50  0000 C CNN
-F 3 "" H 4200 2900 50  0000 C CNN
-	1    4200 2900
+P 4200 3000
+F 0 "C?" H 4225 3100 50  0000 L CNN
+F 1 "CP" H 4225 2900 50  0000 L CNN
+F 2 "" H 4238 2850 50  0000 C CNN
+F 3 "" H 4200 3000 50  0000 C CNN
+	1    4200 3000
 	1    0    0    -1
 $EndComp
@@
 L R R?
 U 1 1 5EACB560
-P 5400 2900
-F 0 "R?" V 5480 2900 50  0000 C CNN
-F 1 "R" V 5400 2900 50  0000 C CNN
-F 2 "" V 5330 2900 50  0000 C CNN
-F 3 "" H 5400 2900 50  0000 C CNN
-	1    5400 2900
+P 5600 2900
+F 0 "R?" V 5680 2900 50  0000 C CNN
+F 1 "R" V 5600 2900 50  0000 C CNN
+F 2 "" V 5530 2900 50  0000 C CNN
+F 3 "" H 5600 2900 50  0000 C CNN
+	1    5600 2900
 	1    0    0    -1
 $EndComp
@@
 L LED D?
 U 1 1 5EACB599
-P 5400 3300
-F 0 "D?" H 5400 3400 50  0000 C CNN
-F 1 "LED" H 5400 3200 50  0000 C CNN
-F 2 "" H 5400 3300 50  0000 C CNN
-F 3 "" H 5400 3300 50  0000 C CNN
-	1    5400 3300
+P 5600 3250
+F 0 "D?" H 5600 3350 50  0000 C CNN
+F 1 "LED" H 5600 3150 50  0000 C CNN
+F 2 "" H 5600 3250 50  0000 C CNN
+F 3 "" H 5600 3250 50  0000 C CNN
+	1    5600 3250
 	0    -1   -1   0
 $EndComp
@@
 L PC817 U?
 U 1 1 5EACB5DE
-P 6200 2800
-F 0 "U?" H 6000 3000 50  0000 L CNN
-F 1 "PC817" H 6200 3000 50  0000 L CNN
-F 2 "DIP-4" H 6000 2600 50  0000 L CIN
-F 3 "" H 6200 2800 50  0000 L CNN
-	1    6200 2800
+P 6300 3100
+F 0 "U?" H 6100 3300 50  0000 L CNN
+F 1 "PC817" H 6300 3300 50  0000 L CNN
+F 2 "DIP-4" H 6100 2900 50  0000 L CIN
+F 3 "" H 6300 3100 50  0000 L CNN
+	1    6300 3100
 	1    0    0    -1
 $EndComp
@@
 L R R?
 U 1 1 5EACB8F3
-P 7100 2250
-F 0 "R?" V 7180 2250 50  0000 C CNN
-F 1 "R" V 7100 2250 50  0000 C CNN
-F 2 "" V 7030 2250 50  0000 C CNN
-F 3 "" H 7100 2250 50  0000 C CNN
-	1    7100 2250
-	1    0    0    -1
-$EndComp
-$Comp
-L GNDREF #PWR?
-U 1 1 5EACB9AA
-P 7100 3650
-F 0 "#PWR?" H 7100 3400 50  0001 C CNN
-F 1 "GNDREF" H 7100 3500 50  0000 C CNN
-F 2 "" H 7100 3650 50  0000 C CNN
-F 3 "" H 7100 3650 50  0000 C CNN
-	1    7100 3650
-	1    0    0    -1
-$EndComp
+P 7100 2600
+F 0 "R?" V 7180 2600 50  0000 C CNN
+F 1 "R" V 7100 2600 50  0000 C CNN
+F 2 "" V 7030 2600 50  0000 C CNN
+F 3 "" H 7100 2600 50  0000 C CNN
+	1    7100 2600
+	1    0    0    -1
+$EndComp
+$Comp
+L Crystal Y?
+U 1 1 5EACBAAE
+P 7450 1000
+F 0 "Y?" H 7450 1150 50  0000 C CNN
+F 1 "Crystal" H 7450 850 50  0000 C CNN
+F 2 "" H 7450 1000 50  0000 C CNN
+F 3 "" H 7450 1000 50  0000 C CNN
+	1    7450 1000
+	1    0    0    -1
+$EndComp
+$Comp
+L R R?
+U 1 1 5EACBB47
+P 7850 1000
+F 0 "R?" V 7930 1000 50  0000 C CNN
+F 1 "R" V 7850 1000 50  0000 C CNN
+F 2 "" V 7780 1000 50  0000 C CNN
+F 3 "" H 7850 1000 50  0000 C CNN
+	1    7850 1000
+	1    0    0    -1
+$EndComp
+$Comp
+L C C?
+U 1 1 5EACBBE0
+P 8150 1000
+F 0 "C?" H 8175 1100 50  0000 L CNN
+F 1 "C" H 8175 900 50  0000 L CNN
+F 2 "" H 8188 850 50  0000 C CNN
+F 3 "" H 8150 1000 50  0000 C CNN
+	1    8150 1000
+	1    0    0    -1
+$EndComp
+$Comp
+L C C?
+U 1 1 5EACBC76
+P 8450 1000
+F 0 "C?" H 8475 1100 50  0000 L CNN
+F 1 "C" H 8475 900 50  0000 L CNN
+F 2 "" H 8488 850 50  0000 C CNN
+F 3 "" H 8450 1000 50  0000 C CNN
+	1    8450 1000
+	1    0    0    -1
+$EndComp
+$Comp
+L C C?
+U 1 1 5EACBCD6
+P 6900 3100
+F 0 "C?" H 6925 3200 50  0000 L CNN
+F 1 "C" H 6925 3000 50  0000 L CNN
+F 2 "" H 6938 2950 50  0000 C CNN
+F 3 "" H 6900 3100 50  0000 C CNN
+	1    6900 3100
+	1    0    0    -1
+$EndComp
+$Comp
+L CP C?
+U 1 1 5EAD6BFF
+P 5300 2900
+F 0 "C?" H 5325 3000 50  0000 L CNN
+F 1 "CP" H 5325 2800 50  0000 L CNN
+F 2 "" H 5338 2750 50  0000 C CNN
+F 3 "" H 5300 2900 50  0000 C CNN
+	1    5300 2900
+	1    0    0    -1
+$EndComp
+$Comp
+L R R?
+U 1 1 5EAD6CA9
+P 5850 2750
+F 0 "R?" V 5930 2750 50  0000 C CNN
+F 1 "R" V 5850 2750 50  0000 C CNN
+F 2 "" V 5780 2750 50  0000 C CNN
+F 3 "" H 5850 2750 50  0000 C CNN
+	1    5850 2750
+	0    1    1    0
+$EndComp
+Wire Wire Line
+	1800 2650 2150 2650
+Wire Wire Line
+	2150 2650 2150 2550
+Wire Wire Line
+	1800 2850 2150 2850
+Wire Wire Line
+	2150 2850 2150 2950
+Wire Wire Line
+	3650 2450 2950 2450
+Wire Wire Line
+	2950 2450 2950 2550
+Wire Wire Line
+	3650 3050 2950 3050
+Wire Wire Line
+	2950 3050 2950 2950
+Wire Wire Line
+	4200 2850 4200 2750
+Wire Wire Line
+	3950 2750 4400 2750
+Connection ~ 4200 2750
+Wire Wire Line
+	3350 2750 3350 3300
+Wire Wire Line
+	3350 3300 5300 3300
+Wire Wire Line
+	4200 3300 4200 3150
+Wire Wire Line
+	4800 3300 4800 3050
+Connection ~ 4200 3300
+Wire Wire Line
+	5200 2750 5700 2750
+Wire Wire Line
+	5300 3050 5300 3400
+Connection ~ 4800 3300
+Connection ~ 5300 2750
+Wire Wire Line
+	5300 3400 6000 3400
+Connection ~ 5300 3300
+Connection ~ 5600 2750
+Wire Wire Line
+	6000 2750 6000 3000
+Wire Wire Line
+	6000 3400 6000 3200
+Connection ~ 5600 3400
+Wire Wire Line
+	5600 3050 5600 3100
+Wire Wire Line
+	6600 2950 7750 2950
+Wire Wire Line
+	6600 2950 6600 3000
+Wire Wire Line
+	6600 3250 7100 3250
+Wire Wire Line
+	6600 3250 6600 3200
+Wire Wire Line
+	7100 3250 7100 3650
+Connection ~ 6900 3250
+Wire Wire Line
+	7100 2300 7100 2450
+Wire Wire Line
+	7100 2950 7100 2750
+Connection ~ 6900 2950
+Wire Wire Line
+	8200 2550 7750 2550
+Wire Wire Line
+	7750 2550 7750 2950
+Connection ~ 7100 2950
+Text Label 7100 2300 0    60   ~ 0
++5v-ATMEGA328P
+Text Label 10100 4350 0    60   ~ 0
++5v-ATMEGA328P
+Text Label 7100 3650 0    60   ~ 0
+GND-ATMEGA328P
+Text Label 10100 2050 0    60   ~ 0
+GND-ATMEGA328P
+Text Notes 7600 2600 0    60   ~ 0
+Digital PIN 2
 $EndSCHEMATC

Commit message: Kicad .sch MAJ
Parts:
- C?: value CP -> 1000uF
- C?: value C -> 10nF
- C?: value CP -> 10uF
- D?: value D_Bridge_-A+A -> Pont de diode
- R? (x2): value R -> 1k
- R?: value R -> 10k
- T?: value Transformer_1P_1S -> Transformer 230v / 12v
Changed lines of the file:
@@
 P 2550 2750
 F 0 "T?" H 2550 3000 50  0000 C CNN
-F 1 "Transformer_1P_1S" H 2550 2450 50  0000 C CNN
+F 1 "Transformer 230v / 12v" H 2550 2450 50  0000 C CNN
 F 2 "" H 2550 2750 50  0000 C CNN
 F 3 "" H 2550 2750 50  0000 C CNN
@@
 P 3650 2750
 F 0 "D?" H 3700 3025 50  0000 L CNN
-F 1 "D_Bridge_-A+A" H 3700 2950 50  0000 L CNN
+F 1 "Pont de diode" H 3700 2950 50  0000 L CNN
 F 2 "" H 3650 2750 50  0000 C CNN
 F 3 "" H 3650 2750 50  0000 C CNN
@@
 P 4200 3000
 F 0 "C?" H 4225 3100 50  0000 L CNN
-F 1 "CP" H 4225 2900 50  0000 L CNN
+F 1 "1000uF" H 4225 2900 50  0000 L CNN
 F 2 "" H 4238 2850 50  0000 C CNN
 F 3 "" H 4200 3000 50  0000 C CNN
@@
 P 5600 2900
 F 0 "R?" V 5680 2900 50  0000 C CNN
-F 1 "R" V 5600 2900 50  0000 C CNN
+F 1 "1k" V 5600 2900 50  0000 C CNN
 F 2 "" V 5530 2900 50  0000 C CNN
 F 3 "" H 5600 2900 50  0000 C CNN
@@
 P 7100 2600
 F 0 "R?" V 7180 2600 50  0000 C CNN
-F 1 "R" V 7100 2600 50  0000 C CNN
+F 1 "10k" V 7100 2600 50  0000 C CNN
 F 2 "" V 7030 2600 50  0000 C CNN
 F 3 "" H 7100 2600 50  0000 C CNN
@@
 P 6900 3100
 F 0 "C?" H 6925 3200 50  0000 L CNN
-F 1 "C" H 6925 3000 50  0000 L CNN
+F 1 "10nF" H 6925 3000 50  0000 L CNN
 F 2 "" H 6938 2950 50  0000 C CNN
 F 3 "" H 6900 3100 50  0000 C CNN
@@
 P 5300 2900
 F 0 "C?" H 5325 3000 50  0000 L CNN
-F 1 "CP" H 5325 2800 50  0000 L CNN
+F 1 "10uF" H 5325 2800 50  0000 L CNN
 F 2 "" H 5338 2750 50  0000 C CNN
 F 3 "" H 5300 2900 50  0000 C CNN
@@
 P 5850 2750
 F 0 "R?" V 5930 2750 50  0000 C CNN
-F 1 "R" V 5850 2750 50  0000 C CNN
+F 1 "1k" V 5850 2750 50  0000 C CNN
 F 2 "" V 5780 2750 50  0000 C CNN
 F 3 "" H 5850 2750 50  0000 C CNN
